Commit message: 修改urdf，导出xml

File: HTDW_5036/urdf/HTDW_5036.urdf (robot description, URDF)
Before this commit: robot HTDW_5036, 17 links, 16 joints
Links:
- link FL_calf: mass 0.18510355836004 -> 0.185104
- link FL_foot: mass 0.0559077087759024 -> 0.051122; geometry collision sphere radius=0.022; visual mesh filename=../meshes/FL_foot.STL
- link FL_hip: mass 0.384243332889522 -> 0.384243
- link FL_thigh: mass 0.474999600734316 -> 0.475
- link FR_calf: mass 0.18510355262369 -> 0.185104
- link FR_foot: mass 0.0559077088519554 -> 0.051122; geometry collision sphere radius=0.022; visual mesh filename=../meshes/FR_foot.STL
- link FR_hip: mass 0.384243332889521 -> 0.384243
- link FR_thigh: mass 0.474999595712705 -> 0.475
- link RL_calf: mass 0.18510355825332 -> 0.185104
- link RL_foot: mass 0.0559077084681938 -> 0.051122; geometry collision sphere radius=0.022; visual mesh filename=../meshes/RL_foot.STL
- link RL_hip: mass 0.384243332889521 -> 0.384243
- link RL_thigh: mass 0.474999600734314 -> 0.475
- link RR_calf: mass 0.185103555370611 -> 0.185104
- link RR_foot: mass 0.0559077088089483 -> 0.051122; geometry collision sphere radius=0.022; visual mesh filename=../meshes/RR_foot.STL
- link RR_hip: mass 0.384243332889522 -> 0.384243
- link RR_thigh: mass 0.474999595712706 -> 0.475
- link base_link: mass 2.69658564891505 -> 2.659586
Joints:
- joint FL_calf_joint: limit lower=-2.65 upper=-0.84 effort=21 velocity=9.5 -> lower=-2.43 upper=-1.298 effort=21 velocity=9.5
- joint FL_foot: origin xyz=-0.00023522 0 -0.18325 rpy=0 0 0 -> xyz=-0.0144485951312854 0 -0.196399042450557 rpy=0 0 0
- joint FR_calf_joint: limit lower=-2.65 upper=-0.84 effort=21 velocity=9.5 -> lower=-2.43 upper=-1.298 effort=21 velocity=9.5
- joint FR_foot: origin xyz=-0.000235191782713057 0 -0.183253819517796 rpy=0 0 0 -> xyz=-0.014449 0 -0.1964 rpy=0 0 0
- joint RL_calf_joint: limit lower=-2.65 upper=-0.84 effort=21 velocity=9.5 -> lower=-2.43 upper=-1.298 effort=21 velocity=9.5
- joint RL_foot: origin xyz=-0.000235191782713084 0 -0.183253819517796 rpy=0 0 0 -> xyz=-0.0144485645043519 0 -0.196399042137075 rpy=0 0 0
- joint RR_calf_joint: limit lower=-2.65 upper=-0.84 effort=21 velocity=9.5 -> lower=-2.43 upper=-1.298 effort=21 velocity=9.5
- joint RR_foot: origin xyz=-0.000235191782713084 0 -0.183253819517796 rpy=0 0 0 -> xyz=-0.0144485645043577 0 -0.196399042137075 rpy=0 0 0
