Commit message: 规范名称问题

File: HTDW_4438/urdf/HTDW_4438.urdf (robot description, URDF)
Before this commit: robot HTDW_4438, 17 links, 16 joints
Links:
- link FL_hip: mass 0.0627632437664346 -> 0.0627632437664345
- link FR_hip: mass 0.0627632437546341 -> 0.0627632437545266
- link RR_thigh: mass 0.264761547961981 -> 0.264761547913784
Joints:
- removed joint FL_foot
- removed joint FR_calf
- removed joint FR_foot_joint
- removed joint RR_calf_joint
- added joint FL_foot_joint: type fixed, parent FL_calf, child FL_foot, origin xyz=0 0 -0.15 rpy=0 0 0, axis 0 0 0
- added joint FR_calf_joint: type revolute, parent FR_thigh, child FR_calf, origin xyz=0 0 -0.15 rpy=0 0 0, axis 0 1 0, limit lower=0 upper=0 effort=0 velocity=0
- added joint FR_foot: type fixed, parent FR_calf, child FR_foot, origin xyz=0 0 -0.15 rpy=0 0 0, axis 0 0 0
- added joint RR_calf: type revolute, parent RR_thigh, child RR_calf, origin xyz=0 0 -0.15 rpy=0 0 0, axis 0 1 0, limit lower=0 upper=0 effort=0 velocity=0
- joint FL_calf_joint: limit lower=-2.53 upper=-0.84 effort=10 velocity=9.5 -> lower=0 upper=0 effort=0 velocity=0
- joint FL_hip_joint: limit lower=-1.05 upper=1.05 effort=10 velocity=9.5 -> lower=0 upper=0 effort=0 velocity=0
- joint FL_thigh_joint: limit lower=-1.57 upper=3.49 effort=10 velocity=9.5 -> lower=0 upper=0 effort=0 velocity=0
- joint FR_hip_joint: limit lower=-1.05 upper=1.05 effort=10 velocity=9.5 -> lower=0 upper=0 effort=0 velocity=0
- joint FR_thigh_joint: limit lower=-1.57 upper=3.49 effort=10 velocity=9.5 -> lower=0 upper=0 effort=0 velocity=0
- joint RL_calf_joint: limit lower=-2.53 upper=-0.84 effort=10 velocity=9.5 -> lower=0 upper=0 effort=0 velocity=0
- joint RL_hip_joint: limit lower=-1.05 upper=1.05 effort=10 velocity=9.5 -> lower=0 upper=0 effort=0 velocity=0
- joint RL_thigh_joint: limit lower=-1.57 upper=3.49 effort=10 velocity=9.5 -> lower=0 upper=0 effort=0 velocity=0
- joint RR_hip_joint: limit lower=-1.05 upper=1.05 effort=10 velocity=9.5 -> lower=0 upper=0 effort=0 velocity=0
- joint RR_thigh_joint: limit lower=-1.57 upper=3.49 effort=10 velocity=9.5 -> lower=0 upper=0 effort=0 velocity=0

Commit message: 上传urdf模型

File: HTDW_4438/urdf/HTDW_4438.urdf (robot description, URDF)
Before this commit: robot HTDW_4438, 17 links, 16 joints
Links:
- link FL_calf: mass 0.153268276445712 -> 0.06068055; geometry collision mesh filename=../meshes/FL_calf.STL; visual mesh filename=../meshes/FL_calf.STL
- link FL_foot: mass 0.0049215011738973 -> 0.0049215; geometry collision sphere radius=0.02; visual mesh filename=../meshes/FL_foot.STL
- link FL_hip: mass 0.0627632437664345 -> 0.27079698; geometry collision mesh filename=../meshes/FL_hip.STL; visual mesh filename=../meshes/FL_hip.STL
- link FL_thigh: mass 0.264760738721982 -> 0.47279447; geometry collision mesh filename=../meshes/FL_thigh.STL; visual mesh filename=../meshes/FL_thigh.STL
- link FR_calf: mass 0.153268271042767 -> 0.06068055; geometry collision mesh filename=../meshes/FR_calf.STL; visual mesh filename=../meshes/FR_calf.STL
- link FR_foot: mass 0.0049215011738973 -> 0.0049215; geometry collision sphere radius=0.02; visual mesh filename=../meshes/FR_foot.STL
- link FR_hip: mass 0.0627632437545266 -> 0.27079698; geometry collision mesh filename=../meshes/FR_hip.STL; visual mesh filename=../meshes/FR_hip.STL
- link FR_thigh: mass 0.264761547925638 -> 0.47279491; geometry collision mesh filename=../meshes/FR_thigh.STL; visual mesh filename=../meshes/FR_thigh.STL
- link RL_calf: mass 0.153268275649899 -> 0.06068055; geometry collision mesh filename=../meshes/RL_calf.STL; visual mesh filename=../meshes/RL_calf.STL
- link RL_foot: mass 0.00492150117389732 -> 0.0049215; geometry collision sphere radius=0.02; visual mesh filename=../meshes/RL_foot.STL
- link RL_hip: mass 0.0627632437669057 -> 0.27079698; geometry collision mesh filename=../meshes/RL_hip.STL; visual mesh filename=../meshes/RL_hip.STL
- link RL_thigh: mass 0.264760738558349 -> 0.47279447; geometry collision mesh filename=../meshes/RL_thigh.STL; visual mesh filename=../meshes/RL_thigh.STL
- link RR_calf: mass 0.153268275552393 -> 0.06068055; geometry collision mesh filename=../meshes/RR_calf.STL; visual mesh filename=../meshes/RR_calf.STL
- link RR_foot: mass 0.00492150117389729 -> 0.0049215; geometry collision sphere radius=0.02; visual mesh filename=../meshes/RR_foot.STL
- link RR_hip: mass 0.0627632437664321 -> 0.27079698; geometry collision mesh filename=../meshes/RR_hip.STL; visual mesh filename=../meshes/RR_hip.STL
- link RR_thigh: mass 0.264761547913784 -> 0.47279491; geometry collision mesh filename=../meshes/RR_thigh.STL; visual mesh filename=../meshes/RR_thigh.STL
- link base_link: mass 1.43623232112764 -> 2.74343032; geometry collision mesh filename=../meshes/base_link.STL; visual mesh filename=../meshes/base_link.STL
Joints:
- joint FL_calf_joint: limit lower=0 upper=0 effort=0 velocity=0 -> lower=-2.53 upper=-0.84 effort=10 velocity=9.5
- joint FL_hip_joint: limit lower=0 upper=0 effort=0 velocity=0 -> lower=-1.05 upper=1.05 effort=10 velocity=9.5
- joint FL_thigh_joint: limit lower=0 upper=0 effort=0 velocity=0 -> lower=-1.57 upper=3.49 effort=10 velocity=9.5
- joint FR_calf_joint: limit lower=0 upper=0 effort=0 velocity=0 -> lower=-2.53 upper=-0.84 effort=10 velocity=9.5
- joint FR_foot: origin xyz=0 0 -0.15 rpy=0 0 0 -> xyz=0 0 -0.149999998990809 rpy=0 0 0
- joint FR_hip_joint: limit lower=0 upper=0 effort=0 velocity=0 -> lower=-1.05 upper=1.05 effort=10 velocity=9.5
- joint FR_thigh_joint: limit lower=0 upper=0 effort=0 velocity=0 -> lower=-1.57 upper=3.49 effort=10 velocity=9.5
- joint RL_calf_joint: limit lower=0 upper=0 effort=0 velocity=0 -> lower=-2.53 upper=-0.84 effort=10 velocity=9.5
- joint RL_hip_joint: limit lower=0 upper=0 effort=0 velocity=0 -> lower=-1.05 upper=1.05 effort=10 velocity=9.5
- joint RL_thigh_joint: limit lower=0 upper=0 effort=0 velocity=0 -> lower=-1.57 upper=3.49 effort=10 velocity=9.5
- joint RR_calf: limit lower=0 upper=0 effort=0 velocity=0 -> lower=-2.53 upper=-0.84 effort=10 velocity=9.5
- joint RR_hip_joint: limit lower=0 upper=0 effort=0 velocity=0 -> lower=-1.05 upper=1.05 effort=10 velocity=9.5
- joint RR_thigh_joint: limit lower=0 upper=0 effort=0 velocity=0 -> lower=-1.57 upper=3.49 effort=10 velocity=9.5

Commit message: 修改urdf模型

File: HTDW_4438/urdf/HTDW_4438.urdf (robot description, URDF)
Before this commit: robot HTDW_4438, 17 links, 16 joints
Links:
- link FL_thigh: mass 0.47279447 -> 0.48086181
- link FR_thigh: mass 0.47279491 -> 0.48086142
- link RL_thigh: mass 0.47279447 -> 0.48086181
- link RR_thigh: mass 0.47279491 -> 0.48086142
Joints:
- removed joint FR_foot
- removed joint RR_calf
- added joint FR_foot_joint: type fixed, parent FR_calf, child FR_foot, origin xyz=-0.017107 0 -0.14902 rpy=0 0 0, axis 0 0 0
- added joint RR_calf_joint: type revolute, parent RR_thigh, child RR_calf, origin xyz=-0.014931 0 -0.14926 rpy=0 0 0, axis 0 1 0, limit lower=-2.53 upper=-0.84 effort=10 velocity=9.5
- joint FL_calf_joint: origin xyz=0 0 -0.15 rpy=0 0 0 -> xyz=-0.0026011 0.0035 -0.14998 rpy=0 0 0
- joint FL_foot_joint: origin xyz=0 0 -0.15 rpy=0 0 0 -> xyz=-0.0026011 0 -0.14998 rpy=0 0 0
- joint FR_calf_joint: origin xyz=0 0 -0.15 rpy=0 0 0 -> xyz=-0.017107 0 -0.14902 rpy=0 0 0
- joint RL_calf_joint: origin xyz=0 0 -0.15 rpy=0 0 0 -> xyz=-0.016035 0 -0.14914 rpy=0 0 0
- joint RL_foot_joint: origin xyz=0 0 -0.15 rpy=0 0 0 -> xyz=-0.0160344934758346 0 -0.149140520034684 rpy=0 0 0
- joint RR_foot_joint: origin xyz=0 0 -0.15 rpy=0 0 0 -> xyz=-0.014931 0 -0.14926 rpy=0 0 0

Commit message: 更正urdf

File: HTDW_4438/urdf/HTDW_4438.urdf (robot description, URDF)
Before this commit: robot HTDW_4438, 17 links, 16 joints
Joints:
- joint FL_calf_joint: origin xyz=-0.0026011 0.0035 -0.14998 rpy=0 0 0 -> xyz=0 0.0035 -0.15 rpy=0 0 0
- joint FL_foot_joint: origin xyz=-0.0026011 0 -0.14998 rpy=0 0 0 -> xyz=0 0 -0.15 rpy=0 0 0
- joint FR_calf_joint: origin xyz=-0.017107 0 -0.14902 rpy=0 0 0 -> xyz=0 0 -0.15 rpy=0 0 0
- joint FR_foot_joint: origin xyz=-0.017107 0 -0.14902 rpy=0 0 0 -> xyz=0 0 -0.15 rpy=0 0 0
- joint RL_calf_joint: origin xyz=-0.016035 0 -0.14914 rpy=0 0 0 -> xyz=0 0 -0.15 rpy=0 0 0
- joint RL_foot_joint: origin xyz=-0.0160344934758346 0 -0.149140520034684 rpy=0 0 0 -> xyz=0 0 -0.15 rpy=0 0 0
- joint RR_calf_joint: origin xyz=-0.014931 0 -0.14926 rpy=0 0 0 -> xyz=0 0 -0.15 rpy=0 0 0
- joint RR_foot_joint: origin xyz=-0.014931 0 -0.14926 rpy=0 0 0 -> xyz=0 0 -0.15 rpy=0 0 0
