Commit message: ri_plus urdf去掉指环

File: ri_plus_4438/urdf/ri_plus_4438.urdf (robot description, URDF)
Before this commit: robot ri_4438, 26 links, 25 joints
Links:
- link gripper_finger_left: mass 0.07421078 -> 0.06406078
- link gripper_finger_right: mass 0.07421078 -> 0.06406078
- link wrist3_link: mass 0.33345013 -> 0.31383978
Joints:
- joint RL_calf_joint: axis 0 1 0 -> 0 -1 0
- joint RL_thigh_joint: axis 0 1 0 -> 0 -1 0
- joint forearm_link_joint: axis 0 1 0 -> 0 -1 0

Commit message: 增加限位

File: ri_plus_4438/urdf/ri_plus_4438.urdf (robot description, URDF)
Before this commit: robot ri_plus_4438, 26 links, 25 joints
Joints:
- joint RL_calf_joint: axis 0 -1 0 -> 0 1 0
