Commit message: 修改电机，修改urdf

File: ri_5036/urdf/ri_5036.urdf (robot description, URDF)
Before this commit: robot ri_5036, 17 links, 16 joints
Links:
- link FL_foot: mass 0.01311889 -> 0.01311792
- link FL_hip: mass 0.37981273 -> 0.20213661
- link FL_thigh: mass 0.57659048 -> 0.40794661
- link FR_foot: mass 0.01311889 -> 0.01311792
- link FR_hip: mass 0.37981273 -> 0.20213661
- link FR_thigh: mass 0.57659026 -> 0.40794627
- link RL_foot: mass 0.01311889 -> 0.01311792
- link RL_hip: mass 0.37981273 -> 0.20213661
- link RL_thigh: mass 0.57659048 -> 0.40794661
- link RR_calf: mass 0.06068055 -> 0.06096356
- link RR_foot: mass 0.01311889 -> 0.01311792
- link RR_hip: mass 0.37981273 -> 0.20213661
- link RR_thigh: mass 0.57659026 -> 0.40794627
- link base_link: mass 2.63602586885978 -> 2.4003459
Joints:
- removed joint FL_calf_Joint
- removed joint FL_foot_Joint
- removed joint FL_hip_Joint
- removed joint FL_thigh_Joint
- removed joint FR_calf_Joint
- removed joint FR_foot_Joint
- removed joint FR_hip_Joint
- removed joint FR_thigh_Joint
- removed joint RL_calf_Joint
- removed joint RL_foot_Joint
- removed joint RL_hip_Joint
- removed joint RL_thigh_Joint
- removed joint RR_calf_Joint
- removed joint RR_foot_Joint
- removed joint RR_hip_Joint
- removed joint RR_thigh_Joint
- added joint FL_calf_joint: type revolute, parent FL_thigh, child FL_calf, origin xyz=0 0 -0.15 rpy=0 0 0, axis 0 1 0, limit lower=-2.7 upper=-0.56 effort=21 velocity=50
- added joint FL_foot_joint: type fixed, parent FL_calf, child FL_foot, origin xyz=0 0 -0.15 rpy=0 0 0, axis 0 0 0
- added joint FL_hip_joint: type revolute, parent base_link, child FL_hip, origin xyz=0.15565 0.041 0 rpy=0 0 0, axis 0 1 0, limit lower=-1.5 upper=1.5 effort=21 velocity=50
- added joint FL_thigh_joint: type revolute, parent FL_hip, child FL_thigh, origin xyz=0 0.1034 0 rpy=0 0 0, axis 0 1 0, limit lower=-1.57 upper=3.49 effort=21 velocity=50
- added joint FR_calf_joint: type revolute, parent FR_thigh, child FR_calf, origin xyz=0 0 -0.15 rpy=0 0 0, axis 0 1 0, limit lower=-2.7 upper=-0.56 effort=21 velocity=50
- added joint FR_foot_joint: type fixed, parent FR_calf, child FR_foot, origin xyz=0 0 -0.15 rpy=0 0 0, axis 0 0 0
- added joint FR_hip_link: type revolute, parent base_link, child FR_hip, origin xyz=0.15564 -0.041 0 rpy=0 0 0, axis 1 0 0, limit lower=-1.5 upper=1.5 effort=21 velocity=50
- added joint FR_thigh_joint: type revolute, parent FR_hip, child FR_thigh, origin xyz=0 -0.1034 0 rpy=0 0 0, axis 0 -1 0, limit lower=-1.57 upper=3.49 effort=21 velocity=50
- added joint RL_calf_joint: type revolute, parent RL_thigh, child RL_calf, origin xyz=0 0 -0.15 rpy=0 0 0, axis 0 1 0, limit lower=-2.7 upper=-0.56 effort=21 velocity=50
- added joint RL_foot_joint: type fixed, parent RL_calf, child RL_foot, origin xyz=0 0 -0.149999998923394 rpy=0 0 0, axis 0 0 0
- added joint RL_hip_joint: type revolute, parent base_link, child RL_hip, origin xyz=-0.15566 0.041 0 rpy=0 0 0, axis 1 0 0, limit lower=-1.5 upper=1.5 effort=21 velocity=50
- added joint RL_thigh_joint: type revolute, parent RL_hip, child RL_thigh, origin xyz=0 0.1034 0 rpy=0 0 0, axis 0 1 0, limit lower=-1.57 upper=3.49 effort=21 velocity=50
- added joint RR_calf_joint: type revolute, parent RR_thigh, child RR_calf, origin xyz=0 0 -0.15 rpy=0 0 0, axis 0 1 0, limit lower=-2.7 upper=-0.56 effort=21 velocity=50
- added joint RR_foot_joint: type fixed, parent RR_calf, child RR_foot, origin xyz=0 0 -0.149999998923393 rpy=0 0 0, axis 0 0 0
- added joint RR_hip_joint: type revolute, parent base_link, child RR_hip, origin xyz=-0.15566 -0.041 0 rpy=0 0 0, axis 1 0 0, limit lower=-1.5 upper=1.5 effort=21 velocity=50
- added joint RR_thigh_joint: type revolute, parent RR_hip, child RR_thigh, origin xyz=0 -0.1034 0 rpy=0 0 0, axis 0 1 0, limit lower=-1.57 upper=3.49 effort=21 velocity=50

File: ri_plus_5036/urdf/ri_plus_5036.urdf (robot description, URDF)
Before this commit: robot ri_plus_5036, 26 links, 25 joints
Links:
- link FL_hip: mass 0.37981273 -> 0.20213661
- link FL_thigh: mass 0.57659048 -> 0.40794661
- link FR_hip: mass 0.37981273 -> 0.20213661
- link FR_thigh: mass 0.57659026 -> 0.40794627
- link RL_hip: mass 0.37981273 -> 0.20213661
- link RL_thigh: mass 0.57659048 -> 0.40794661
- link RR_calf: mass 0.06068055 -> 0.06096356
- link RR_hip: mass 0.37981273 -> 0.20213661
- link RR_thigh: mass 0.57659026 -> 0.40794627
- link base_link: mass 3.11108908 -> 2.4003459
Joints:
- joint FL_hip_joint: origin xyz=0.15065 0.041 0 rpy=0 0 0 -> xyz=0.15565 0.041 0 rpy=0 0 0
- joint FL_thigh_joint: origin xyz=0 0.0933 0 rpy=0 0 0 -> xyz=0 0.1034 0 rpy=0 0 0
- joint FR_hip_link: origin xyz=0.15065 -0.041 0 rpy=0 0 0 -> xyz=0.15564 -0.041 0 rpy=0 0 0
- joint FR_thigh_joint: axis 0 1 0 -> 0 -1 0; limit lower=1.57 upper=3.49 effort=21 velocity=50 -> lower=-1.57 upper=3.49 effort=21 velocity=50; origin xyz=0 -0.0933 0 rpy=0 0 0 -> xyz=0 -0.1034 0 rpy=0 0 0
- joint RL_hip_joint: origin xyz=-0.15065 0.041 0 rpy=0 0 0 -> xyz=-0.15566 0.041 0 rpy=0 0 0
- joint RL_thigh_joint: origin xyz=0 0.0933 0 rpy=0 0 0 -> xyz=0 0.1034 0 rpy=0 0 0
- joint RR_foot_joint: origin xyz=0 0 -0.149999998990809 rpy=0 0 0 -> xyz=0 0 -0.149999998923393 rpy=0 0 0
- joint RR_hip_joint: origin xyz=-0.15065 -0.041 0 rpy=0 0 0 -> xyz=-0.15566 -0.041 0 rpy=0 0 0
- joint RR_thigh_joint: origin xyz=0 -0.0933 0 rpy=0 0 0 -> xyz=0 -0.1034 0 rpy=0 0 0

Commit message: 修改连接块

File: ri_5036/urdf/ri_5036.urdf (robot description, URDF)
Before this commit: robot ri_5036, 17 links, 16 joints
Joints:
- joint FR_thigh_joint: axis 0 -1 0 -> 0 1 0
- joint RL_foot_joint: origin xyz=0 0 -0.149999998923394 rpy=0 0 0 -> xyz=0 0 -0.15 rpy=0 0 0
- joint RR_foot_joint: origin xyz=0 0 -0.149999998923393 rpy=0 0 0 -> xyz=0 0 -0.15 rpy=0 0 0

File: ri_plus_5036/urdf/ri_plus_5036.urdf (robot description, URDF)
Before this commit: robot ri_plus_5036, 26 links, 25 joints
Joints:
- joint FL_foot_joint: origin xyz=0 0 -0.15 rpy=0 0 0 -> xyz=0 0 -0.149999998923393 rpy=0 0 0
- joint FR_foot_joint: origin xyz=0 0 -0.15 rpy=0 0 0 -> xyz=0 0 -0.149999998923393 rpy=0 0 0
- joint FR_thigh_joint: axis 0 -1 0 -> 0 1 0

Commit message: 修改腿部比例，更换连杆轴承，修改对应URDF

File: ri_5036/urdf/ri_5036.urdf (robot description, URDF)
Before this commit: robot ri_5036, 17 links, 16 joints
Links:
- link FL_calf: mass 0.06068055 -> 0.0779043
- link FL_foot: mass 0.01311792 -> 0.01311889; geometry collision sphere radius=0.01675; visual mesh filename=../meshes/FL_foot.STL
- link FL_hip: mass 0.20213661 -> 0.19699252
- link FL_thigh: mass 0.40794661 -> 0.45986342
- link FR_calf: mass 0.06068055 -> 0.0779043
- link FR_foot: mass 0.01311792 -> 0.01311889; geometry collision sphere radius=0.01675; visual mesh filename=../meshes/FR_foot.STL
- link FR_hip: mass 0.20213661 -> 0.19699252
- link FR_thigh: mass 0.40794627 -> 0.45512966
- link RL_calf: mass 0.06068055 -> 0.0779043
- link RL_foot: mass 0.01311792 -> 0.01311889; geometry collision sphere radius=0.01675; visual mesh filename=../meshes/RL_foot.STL
- link RL_hip: mass 0.20213661 -> 0.19699252
- link RL_thigh: mass 0.40794661 -> 0.45986342
- link RR_calf: mass 0.06096356 -> 0.0779043
- link RR_foot: mass 0.01311792 -> 0.01311889; geometry collision sphere radius=0.01675; visual mesh filename=../meshes/RR_foot.STL
- link RR_hip: mass 0.20213661 -> 0.19699252
- link RR_thigh: mass 0.40794627 -> 0.45512966
- link base_link: mass 2.4003459 -> 1.52043836128824
Joints:
- removed joint FR_hip_link
- added joint FR_hip_joint: type revolute, parent base_link, child FR_hip, origin xyz=0.15216 -0.041 0 rpy=0 0 0, axis 1 0 0, limit lower=-1.5 upper=1.5 effort=21 velocity=50
- joint FL_calf_joint: origin xyz=0 0 -0.15 rpy=0 0 0 -> xyz=0 0 -0.16 rpy=0 0 0
- joint FL_foot_joint: origin xyz=0 0 -0.15 rpy=0 0 0 -> xyz=0 0 -0.16 rpy=0 0 0
- joint FL_hip_joint: origin xyz=0.15565 0.041 0 rpy=0 0 0 -> xyz=0.15215 0.041 0 rpy=0 0 0
- joint FL_thigh_joint: origin xyz=0 0.1034 0 rpy=0 0 0 -> xyz=0 0.0999 0 rpy=0 0 0
- joint FR_calf_joint: origin xyz=0 0 -0.15 rpy=0 0 0 -> xyz=0 0 -0.16 rpy=0 0 0
- joint FR_foot_joint: origin xyz=0 0 -0.15 rpy=0 0 0 -> xyz=0 0 -0.16 rpy=0 0 0
- joint FR_thigh_joint: limit lower=-1.57 upper=3.49 effort=21 velocity=50 -> lower=1.57 upper=3.49 effort=21 velocity=50; origin xyz=0 -0.1034 0 rpy=0 0 0 -> xyz=0 -0.0999 0 rpy=0 0 0
- joint RL_calf_joint: origin xyz=0 0 -0.15 rpy=0 0 0 -> xyz=0 0 -0.16 rpy=0 0 0
- joint RL_foot_joint: origin xyz=0 0 -0.15 rpy=0 0 0 -> xyz=0 0 -0.16 rpy=0 0 0
- joint RL_hip_joint: origin xyz=-0.15566 0.041 0 rpy=0 0 0 -> xyz=-0.15216 0.041 0 rpy=0 0 0
- joint RL_thigh_joint: origin xyz=0 0.1034 0 rpy=0 0 0 -> xyz=0 0.0999 0 rpy=0 0 0
- joint RR_calf_joint: origin xyz=0 0 -0.15 rpy=0 0 0 -> xyz=0 0 -0.16 rpy=0 0 0
- joint RR_foot_joint: origin xyz=0 0 -0.15 rpy=0 0 0 -> xyz=0 0 -0.16 rpy=0 0 0
- joint RR_hip_joint: origin xyz=-0.15566 -0.041 0 rpy=0 0 0 -> xyz=-0.15214 -0.041 0 rpy=0 0 0
- joint RR_thigh_joint: origin xyz=0 -0.1034 0 rpy=0 0 0 -> xyz=0 -0.0999 0 rpy=0 0 0

File: ri_plus_5036/urdf/ri_plus_5036.urdf (robot description, URDF)
Before this commit: robot ri_plus_5036, 26 links, 25 joints
Links:
- link FL_calf: mass 0.06068055 -> 0.0779043
- link FL_thigh: mass 0.40794661 -> 0.45986342
- link FR_calf: mass 0.06068055 -> 0.0779043
- link FR_thigh: mass 0.40794627 -> 0.45512966
- link RL_calf: mass 0.06068055 -> 0.0779043
- link RL_thigh: mass 0.40794661 -> 0.45986342
- link RR_calf: mass 0.06096356 -> 0.0779043
- link RR_thigh: mass 0.40794627 -> 0.45512966
Joints:
- joint FL_calf_joint: origin xyz=0 0 -0.15 rpy=0 0 0 -> xyz=0 0 -0.16 rpy=0 0 0
- joint FL_foot_joint: origin xyz=0 0 -0.149999998923393 rpy=0 0 0 -> xyz=0 0 -0.16 rpy=0 0 0
- joint FL_hip_joint: origin xyz=0.15565 0.041 0 rpy=0 0 0 -> xyz=0.15215 0.041 0 rpy=0 0 0
- joint FL_thigh_joint: origin xyz=0 0.1034 0 rpy=0 0 0 -> xyz=0 0.0999 0 rpy=0 0 0
- joint FR_calf_joint: origin xyz=0 0 -0.15 rpy=0 0 0 -> xyz=0 0 -0.16 rpy=0 0 0
- joint FR_foot_joint: origin xyz=0 0 -0.149999998923393 rpy=0 0 0 -> xyz=0 0 -0.159999999999985 rpy=0 0 0
- joint FR_hip_link: origin xyz=0.15564 -0.041 0 rpy=0 0 0 -> xyz=0.15216 -0.041 0 rpy=0 0 0
- joint FR_thigh_joint: origin xyz=0 -0.1034 0 rpy=0 0 0 -> xyz=0 -0.0999 0 rpy=0 0 0
- joint RL_calf_joint: origin xyz=0 0 -0.15 rpy=0 0 0 -> xyz=0 0 -0.16 rpy=0 0 0
- joint RL_foot_joint: origin xyz=0 0 -0.15 rpy=0 0 0 -> xyz=0 0 -0.16 rpy=0 0 0
- joint RL_hip_joint: origin xyz=-0.15566 0.041 0 rpy=0 0 0 -> xyz=-0.15216 0.041 0 rpy=0 0 0
- joint RL_thigh_joint: origin xyz=0 0.1034 0 rpy=0 0 0 -> xyz=0 0.0999 0 rpy=0 0 0
- joint RR_calf_joint: origin xyz=0 0 -0.15 rpy=0 0 0 -> xyz=0 0 -0.16 rpy=0 0 0
- joint RR_foot_joint: origin xyz=0 0 -0.149999998923393 rpy=0 0 0 -> xyz=0 0 -0.16 rpy=0 0 0
- joint RR_hip_joint: origin xyz=-0.15566 -0.041 0 rpy=0 0 0 -> xyz=-0.15214 -0.041 0 rpy=0 0 0
- joint RR_thigh_joint: origin xyz=0 -0.1034 0 rpy=0 0 0 -> xyz=0 -0.0999 0 rpy=0 0 0
- joint gripper_finger_left_joint: origin xyz=0.06925 0 0 rpy=0 0 0 -> xyz=0.0692500000000068 0 0 rpy=0 0 0
- joint gripper_finger_right_joint: origin xyz=0.06925 0 0 rpy=0 0 0 -> xyz=0.0692500000000068 0 0 rpy=0 0 0

Commit message: 更换新版电机，修改模型和urdf

File: ri_5036/urdf/ri_5036.urdf (robot description, URDF)
Before this commit: robot ri_5036, 17 links, 16 joints
Links:
- link FL_calf: mass 0.0779043 -> 0.08691043
- link FL_foot: mass 0.01311889 -> 0.01517652; geometry collision mesh filename=../meshes/FL_foot.STL; visual mesh filename=../meshes/FL_foot.STL
- link FL_hip: mass 0.19699252 -> 0.2146778
- link FL_thigh: mass 0.45986342 -> 0.61626132
- link FR_calf: mass 0.0779043 -> 0.08691043
- link FR_foot: mass 0.01311889 -> 0.01517652; geometry collision mesh filename=../meshes/FR_foot.STL; visual mesh filename=../meshes/FR_foot.STL
- link FR_hip: mass 0.19699252 -> 0.2146778
- link FR_thigh: mass 0.45512966 -> 0.61625734
- link RL_calf: mass 0.0779043 -> 0.08691043
- link RL_foot: mass 0.01311889 -> 0.01517652; geometry collision mesh filename=../meshes/RL_foot.STL; visual mesh filename=../meshes/RL_foot.STL
- link RL_hip: mass 0.19699252 -> 0.2146778
- link RL_thigh: mass 0.45986342 -> 0.61626132
- link RR_calf: mass 0.0779043 -> 0.08691043
- link RR_foot: mass 0.01311889 -> 0.01517652; geometry collision mesh filename=../meshes/RR_foot.STL; visual mesh filename=../meshes/RR_foot.STL
- link RR_hip: mass 0.19699252 -> 0.2146778
- link RR_thigh: mass 0.45512966 -> 0.61625734
- link base_link: mass 1.52043836128824 -> 2.43201843
Joints:
- removed joint FR_hip_joint
- added joint FR_hip_link: type revolute, parent base_link, child FR_hip, origin xyz=0.15136 -0.041 0 rpy=0 0 0, axis 1 0 0, limit lower=-1.5 upper=1.5 effort=21 velocity=50
- joint FL_calf_joint: origin xyz=0 0 -0.16 rpy=0 0 0 -> xyz=0 0 -0.2 rpy=0 0 0
- joint FL_foot_joint: origin xyz=0 0 -0.16 rpy=0 0 0 -> xyz=0 0 -0.2 rpy=0 0 0
- joint FL_hip_joint: axis 0 1 0 -> 1 0 0; origin xyz=0.15215 0.041 0 rpy=0 0 0 -> xyz=0.15137 0.041 0 rpy=0 0 0
- joint FL_thigh_joint: origin xyz=0 0.0999 0 rpy=0 0 0 -> xyz=0 0.092718 0 rpy=0 0 0
- joint FR_calf_joint: origin xyz=0 0 -0.16 rpy=0 0 0 -> xyz=0 0 -0.2 rpy=0 0 0
- joint FR_foot_joint: origin xyz=0 0 -0.16 rpy=0 0 0 -> xyz=0 0 -0.2 rpy=0 0 0
- joint FR_thigh_joint: limit lower=1.57 upper=3.49 effort=21 velocity=50 -> lower=-1.57 upper=3.49 effort=21 velocity=50; origin xyz=0 -0.0999 0 rpy=0 0 0 -> xyz=0 -0.092718 0 rpy=0 0 0
- joint RL_calf_joint: origin xyz=0 0 -0.16 rpy=0 0 0 -> xyz=0 0 -0.2 rpy=0 0 0
- joint RL_foot_joint: origin xyz=0 0 -0.16 rpy=0 0 0 -> xyz=0 0 -0.2 rpy=0 0 0
- joint RL_hip_joint: origin xyz=-0.15216 0.041 0 rpy=0 0 0 -> xyz=-0.15137 0.041 0 rpy=0 0 0
- joint RL_thigh_joint: origin xyz=0 0.0999 0 rpy=0 0 0 -> xyz=0 0.092718 0 rpy=0 0 0
- joint RR_calf_joint: origin xyz=0 0 -0.16 rpy=0 0 0 -> xyz=0 0 -0.2 rpy=0 0 0
- joint RR_foot_joint: origin xyz=0 0 -0.16 rpy=0 0 0 -> xyz=0 0 -0.2 rpy=0 0 0
- joint RR_hip_joint: origin xyz=-0.15214 -0.041 0 rpy=0 0 0 -> xyz=-0.15137 -0.041 0 rpy=0 0 0
- joint RR_thigh_joint: origin xyz=0 -0.0999 0 rpy=0 0 0 -> xyz=0 -0.092718 0 rpy=0 0 0
